File: Circuit Design/Circuit_v1/Circuit_v1.kicad_sch (KiCad schematic)
At the start: 0 parts

Commit message: Add controller schematic (KiCad 10) for Spin Coater v1
Fills the empty Circuit_v1.kicad_sch with the full controller wiring:
12V input with 1000uF bulk cap, 1N4007 + 12V->5V buck, SimonK 30A ESC and
A2212 motor, ESP32 DevKit V1 (30-pin DOIT), SSD1306 OLED, 4x4 keypad,
tachometer and E-stop with the 10k pull-ups GPIO34/35 need, and an
optional NPN buzzer driver.

Nets follow firmware/include/config.h and firmware/CIRCUIT.md. Custom
symbols live in the project library spincoater.kicad_sym (sym-lib-table).
ERC: 0 errors, 0 warnings (kicad-cli 10.0.7, all severities).
.kicad_pro and .kicad_pcb are unchanged.
Parts:
- added BZ1: Active buzzer 5V, symbol Device:Buzzer
- added C1: 1000uF 25V, symbol Device:C_Polarized
- added C2: 100nF, symbol Device:C
- added D1: 1N4007, symbol Device:D
- added D2: 1N4148, symbol Device:D
- added J1: 12V IN (SMPS), symbol Connector_Generic:Conn_01x02
- added KP1: 4x4 membrane keypad, symbol spincoater:Keypad_4x4
- added M1: A2212 1400KV, symbol spincoater:BLDC_Motor
- added Q1: 2N2222, symbol Device:Q_NPN
- added R1, R2: 10k, symbol Device:R
- added R3: 1k, symbol Device:R
- added SW1: E-STOP (NO), symbol Switch:SW_Push
- added U1: ESP32 DevKit V1 (CP2102), symbol spincoater:ESP32_DevKit_V1
- added U2: Buck 12V->5V 5A (set 5.0V), symbol spincoater:Buck_Module
- added U3: SimonK 30A ESC, symbol spincoater:SimonK_ESC_30A
- added U4: SSD1306 0.96in I2C (0x3C), symbol spincoater:SSD1306_OLED_I2C
- added U5: IR/Hall tach (1 pulse/rev), symbol spincoater:Tach_Sensor
Connections:
- new net: M1.1 (A), U3.6 (A)
- new net: M1.2 (B), U3.7 (B)
- new net: M1.3 (C), U3.8 (C)
- new net +12V: C1.1, D1.2 (A), J1.1 (Pin_1), U3.1 (V+)
- new net +3V3: R1.1, R2.1, U1.30 (3V3), U5.1 (VCC)
- new net +5V: BZ1.1 (+), C2.1, D2.1 (K), U1.15 (VIN), U2.3 (VOUT+), U4.2 (VCC)
- new net BUZZER: R3.1, U1.16 (GPIO23)
- new net BZ_BASE: Q1.B, R3.2
- new net BZ_DRV: BZ1.2 (-), D2.2 (A), Q1.C
- new net ESC_SIG: U1.13 (GPIO13), U3.3 (SIG)
- new net ESTOP: R2.2, SW1.1, U1.5 (GPIO35)
- new net GND: C1.2, C2.2, J1.2 (Pin_2), Q1.E, SW1.2, U1.14 (GND), U1.29 (GND), U2.2 (VIN-), U2.4 (VOUT-), U3.2 (V-), U3.4 (GND), U4.1 (GND), U5.2 (GND)
- new net KP_C1: KP1.5 (C1), U1.7 (GPIO33)
- new net KP_C2: KP1.6 (C2), U1.6 (GPIO32)
- new net KP_C3: KP1.7 (C3), U1.22 (GPIO18)
- new net KP_C4: KP1.8 (C4), U1.21 (GPIO19)
- new net KP_R1: KP1.1 (R1), U1.11 (GPIO14)
- new net KP_R2: KP1.2 (R2), U1.10 (GPIO27)
- new net KP_R3: KP1.3 (R3), U1.9 (GPIO26)
- new net KP_R4: KP1.4 (R4), U1.8 (GPIO25)
- new net SCL: U1.17 (GPIO22), U4.3 (SCL)
- new net SDA: U1.20 (GPIO21), U4.4 (SDA)
- new net TACH: R1.2, U1.4 (GPIO34), U5.3 (OUT)
- new net VBUCK_IN: D1.1 (K), U2.1 (VIN+)
- no-connect marks 0 -> 13
Other:
- note added: "12V POWER IN + LOGIC 5V"
- note added: "Buzzer optional (firmware does not drive it yet). D2: flyback diode across the buzzer."
- note added: "C1: solder right at the ESC V+/V- input"
- note added: "C2: at ESP32 VIN/GND pins"
- note added: "ESC BEC 5V lead: tape off, do NOT connect. Motor phases: any order, swap two to reverse."
- note added: "ESP32 DEVKIT V1 (CP2102)"
- note added: "Header pins: DOIT 30-pin silkscreen order. Clones vary: wire by the GPIO label on the board. GPIO36 (VP) reserved for an optional current sensor."
- note added: "Keypad rows use the ESP32 internal pull-ups: no resistors. Verify R/C pins with continuity."
- note added: "MOTOR POWER (12V, 14-16 AWG, never on breadboard)"
- note added: "R1 required: GPIO34 has no internal pull-up (omit only if the module has one). Firmware: USE_TACHO 1"
- note added: "R2 required: GPIO35 has no internal pull-up. NO button: ESTOP_ACTIVE_LEVEL LOW. Firmware: USE_ESTOP_PIN 1"
- note added: "TACH + E-STOP + BUZZER"
- note added: "UI: OLED + KEYPAD"
- note added: "WIRING RULES (firmware/CIRCUIT.md) - Mains L/N/Earth into the 12V 15A SMPS is not shown. Earth the SMPS case; switch on Live. - +12V, ESC V+/V- and motor phases: thick wire, XT60/bullets, never through the breadboard. - Star ground near buck VOUT-: SMPS -, buck -, ESC signal GND, ESP32 GND, OLED, tach, E-stop. - Set the buck to 5.0V before connecting the ESP32. ESC BEC 5V stays unconnected. - USB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"
- title: (none) -> Spin Coater v1 - Controller wiring
